File: hardware/kicad/DEVid-Buzz.kicad_sch (KiCad schematic)
At the start: 14 parts, among them SW5 SW_DIP_x04, SW6 SW_DIP_x04, U5 74HC165

Commit message: chore: KiCad 회로도 최신 변경사항 반영
원본 작업 폴더가 "회로도 편집 완료/20260901_ver01"로 재구성됨(이전 smartvault-pcb-1
경로는 더 이상 존재하지 않음). 하위 시트 6개 전부와 최상위 시트에 실제 설계 변경
있음(DoorRock-drv는 축소, 최상위 시트는 대폭 확장 — 회로가 재구성된 것으로 보임).
PCB 레이아웃 자체는 변경 없음. footprint.xlsx(부품-풋프린트 매핑) 신규 추가.

파일 내부의 프로젝트명 자기참조는 원본 작업 파일명("20260901_ver01")이 아니라
저장소 표준 이름("smartvault")으로 맞춰서 복사 — 작업 폴더 쪽 날짜/버전 파일명
관례를 저장소까지 끌고 오지 않음(git이 버전을 관리).

s_vault.kicad_sym(커스텀 심볼 라이브러리)은 원본 경로에서 찾지 못해 갱신 못함 —
RS485-com/power 시트가 이 라이브러리를 참조하므로, 최신 심볼이 바뀌었다면 다음에
갱신 필요(hardware/README.md에 기록해둠).

Co-Authored-By: Claude Sonnet 5 <noreply@anthropic.com>
Parts:
- removed JP1: Jumper_2_Bridged, symbol Jumper:Jumper_2_Bridged
- BZ1: footprint (none) -> Buzzer_Beeper:Buzzer_15x7.5RM7.6
- R12, R14, R15, R16, R17, R18, R19, R20, R21: footprint (none) -> Resistor_SMD:R_0805_2012Metric
Connections:
- net 5V_PULL_UP is gone; now on net 5V_RAW: R14.1, R15.1, R16.1, R17.1, R18.1, R19.1, R20.1, R21.1
- net 5V_RAW: now reaches U5.16 (VCC)
- net Arduino_D7: now reaches R12.1
- net A4_INO renamed Arduino_A3
- net D13_INO renamed Arduino_A5
- net D9_INO renamed Arduino_A4
