File: hardware/kicad/MFRC522_Conn.kicad_sch (KiCad schematic)
At the start: 31 parts, among them U6 74LVC138A, U7 74LVC138A, U8 74LVC125A, U9 74AHCT1G125

Commit message: chore: KiCad 회로도 최신 변경사항 반영
원본 작업 폴더가 "회로도 편집 완료/20260901_ver01"로 재구성됨(이전 smartvault-pcb-1
경로는 더 이상 존재하지 않음). 하위 시트 6개 전부와 최상위 시트에 실제 설계 변경
있음(DoorRock-drv는 축소, 최상위 시트는 대폭 확장 — 회로가 재구성된 것으로 보임).
PCB 레이아웃 자체는 변경 없음. footprint.xlsx(부품-풋프린트 매핑) 신규 추가.

파일 내부의 프로젝트명 자기참조는 원본 작업 파일명("20260901_ver01")이 아니라
저장소 표준 이름("smartvault")으로 맞춰서 복사 — 작업 폴더 쪽 날짜/버전 파일명
관례를 저장소까지 끌고 오지 않음(git이 버전을 관리).

s_vault.kicad_sym(커스텀 심볼 라이브러리)은 원본 경로에서 찾지 못해 갱신 못함 —
RS485-com/power 시트가 이 라이브러리를 참조하므로, 최신 심볼이 바뀌었다면 다음에
갱신 필요(hardware/README.md에 기록해둠).

Co-Authored-By: Claude Sonnet 5 <noreply@anthropic.com>
Parts:
- C11, C12, C13, C14: footprint (none) -> Capacitor_SMD:C_0805_2012Metric
- J_MFC_1, J_MFC_10, J_MFC_2, J_MFC_3, J_MFC_4, J_MFC_5, J_MFC_6, J_MFC_7, J_MFC_8, J_MFC_9: footprint (none) -> Connector_PinSocket_2.54mm:PinSocket_1x08_P2.54mm_Vertical
- R13, R22, R23, R25, R26, R27, R28, R29, R30, R31, R32, R33, R34: footprint (none) -> Resistor_SMD:R_0805_2012Metric
Connections:
- net Arduino_D9: no longer U9.4
- new net Arduino_12: U9.4
Changed lines of the file:
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@@
 	)
 	(junction
+		(at 50.8 121.92)
+		(diameter 0)
+		(color 0 0 0 0)
+	)
+	(junction
 		(at 113.03 156.21)
 		(diameter 0)
@@
 	)
 	(junction
-		(at 50.8 121.92)
-		(diameter 0)
-		(color 0 0 0 0)
-	)
-	(junction
 		(at 87.63 121.92)
 		(diameter 0)
@@
 	)
 	(image
-		(at -74.93 189.23)
-		(scale 1.80766)
+		(at -208.28 90.17)
+		(scale 5.78839)
 		(data "iVBORw0KGgoAAAANSUhEUgAAAyAAAAKiCAYAAAAuf7gPAAAABHNCSVQICAgIfAhkiAAAIABJREFU"
 			"eJzsnXl8FOX9+N8zO7ubbO6LhCQEiICGQ+4bEasgKipVFBCoBdGK8aqK2OrX+6gtLVJsvypiLdaK"
@@
 		)
 	)
-	(label "DEC_A"
-		(at 45.72 121.92 180)
-		(effects
-			(font
-				(size 1.27 1.27)
-			)
-			(justify right bottom)
-		)
-	)
 	(label "MOSI_3V3"
 		(at 257.81 83.82 270)
@@
 		)
 	)
-	(label "DEC_C"
-		(at 45.72 127 180)
-		(effects
-			(font
-				(size 1.27 1.27)
-			)
-			(justify right bottom)
-		)
-	)
 	(label "+3V3"
 		(at 172.72 83.82 270)
@@
 		)
 	)
-	(label "DEC_B"
-		(at 45.72 124.46 180)
-		(effects
-			(font
-				(size 1.27 1.27)
-			)
-			(justify right bottom)
-		)
-	)
 	(label ""
 		(at 232.41 41.91 0)
@@
 		(shape input)
 		(at 30.48 127 180)
-		(fields_autoplaced yes)
 		(effects
 			(font
@@
 			)
 		)
+		(property "Netclass" "Default"
+			(at 30.48 130.8418 0)
+			(hide yes)
+			(show_name no)
+			(do_not_autoplace no)
+			(effects
+				(font
+					(size 1.27 1.27)
+				)
+				(justify right)
+			)
+		)
+		(property "필드" "DEC_C"
+			(at 47.244 125.984 0)
+			(show_name no)
+			(do_not_autoplace no)
+			(effects
+				(font
+					(size 1.27 1.27)
+				)
+				(justify right)
+			)
+		)
 	)
 	(global_label "3V3_RAW"
@@
 		)
 	)
-	(global_label "Arduino_D9"
-		(shape input)
-		(at 54.61 67.31 180)
-		(fields_autoplaced yes)
-		(effects
-			(font
-				(size 1.27 1.27)
-			)
-			(justify right)
-		)
-		(property "Intersheetrefs" "${INTERSHEET_REFS}"
-			(at 41.1021 67.31 0)
-			(hide yes)
-			(show_name no)
-			(do_not_autoplace no)
-			(effects
-				(font
-					(size 1.27 1.27)
-				)
-				(justify right)
-			)
-		)
-	)
 	(global_label "3V3_RAW"
 		(shape input)
@@
 		)
 	)
-	(global_label "Arduino_D9"
+	(global_label "Arduino_12"
 		(shape output)
 		(at 54.61 96.52 180)
@@
 		)
 		(property "Intersheetrefs" "${INTERSHEET_REFS}"
-			(at 41.1021 96.52 0)
+			(at 41.1626 96.52 0)
 			(hide yes)
 			(show_name no)
@@
 		)
 	)
+	(global_label "Arduino_D9"
+		(shape input)
+		(at 54.61 67.31 180)
+		(fields_autoplaced yes)
+		(effects
+			(font
+				(size 1.27 1.27)
+			)
+			(justify right)
+		)
+		(property "Intersheetrefs" "${INTERSHEET_REFS}"
+			(at 41.1021 67.31 0)
+			(hide yes)
+			(show_name no)
+			(do_not_autoplace no)
+			(effects
+				(font
+					(size 1.27 1.27)
+				)
+				(justify right)
+			)
+		)
+		(property "Netclass" "Default"
+			(at 54.61 71.1518 0)
+			(hide yes)
+			(show_name no)
+			(do_not_autoplace no)
+			(effects
+				(font
+					(size 1.27 1.27)
+				)
+				(justify right)
+			)
+		)
+		(property "필드" ""
+			(at 54.61 71.1518 0)
+			(hide yes)
+			(show_name no)
+			(do_not_autoplace no)
+			(effects
+				(font
+					(size 1.27 1.27)
+				)
+				(justify right)
+			)
+		)
+	)
 	(global_label "Arduino_D2"
 		(shape input)
 		(at 30.48 121.92 180)
-		(fields_autoplaced yes)
 		(effects
 			(font
@@
 			)
 		)
+		(property "Netclass" "Default"
+			(at 30.48 125.7618 0)
+			(hide yes)
+			(show_name no)
+			(do_not_autoplace no)
+			(effects
+				(font
+					(size 1.27 1.27)
+				)
+				(justify right)
+			)
+		)
+		(property "필드" "DEC_A"
+			(at 46.99 120.65 0)
+			(show_name no)
+			(do_not_autoplace no)
+			(effects
+				(font
+					(size 1.27 1.27)
+				)
+				(justify right)
+			)
+		)
 	)
 	(global_label "3V3_RAW"
@@
 		(shape input)
 		(at 30.48 124.46 180)
-		(fields_autoplaced yes)
 		(effects
 			(font
@@
 			)
 		)
+		(property "Netclass" "Default"
+			(at 30.48 128.3018 0)
+			(hide yes)
+			(show_name no)
+			(do_not_autoplace no)
+			(effects
+				(font
+					(size 1.27 1.27)
+				)
+				(justify right)
+			)
+		)
+		(property "필드" "DEC_B"
+			(at 47.244 123.444 0)
+			(show_name no)
+			(do_not_autoplace no)
+			(effects
+				(font
+					(size 1.27 1.27)
+				)
+				(justify right)
+			)
+		)
 	)
 	(global_label "3V3_RAW"
@@
 			)
 		)
-		(property "Footprint" ""
+		(property "Footprint" "Connector_PinSocket_2.54mm:PinSocket_1x08_P2.54mm_Vertical"
 			(at 236.22 78.74 0)
 			(hide yes)
@@
 			)
 		)
-		(property "Footprint" ""
+		(property "Footprint" "Resistor_SMD:R_0805_2012Metric"
 			(at 100.33 50.038 90)
 			(hide yes)
@@
 			)
 		)
-		(property "Footprint" ""
+		(property "Footprint" "Resistor_SMD:R_0805_2012Metric"
 			(at 91.44 128.778 90)
 			(hide yes)
@@
 			)
 		)
-		(property "Footprint" ""
+		(property "Footprint" "Connector_PinSocket_2.54mm:PinSocket_1x08_P2.54mm_Vertical"
 			(at 237.49 34.29 0)
 			(hide yes)
@@
 			)
 		)
-		(property "Footprint" ""
+		(property "Footprint" "Resistor_SMD:R_0805_2012Metric"
 			(at 100.33 32.258 90)
 			(hide yes)
@@
 			)
 		)
-		(property "Footprint" ""
+		(property "Footprint" "Resistor_SMD:R_0805_2012Metric"
 			(at 91.44 126.238 90)
 			(hide yes)
@@
 			)
 		)
-		(property "Footprint" ""
+		(property "Footprint" "Resistor_SMD:R_0805_2012Metric"
 			(at 91.44 123.698 90)
 			(hide yes)
@@
 			)
 		)
-		(property "Footprint" ""
+		(property "Footprint" "Resistor_SMD:R_0805_2012Metric"
 			(at 91.44 131.318 90)
 			(hide yes)
@@
 			)
 		)
-		(property "Footprint" ""
+		(property "Footprint" "Connector_PinSocket_2.54mm:PinSocket_1x08_P2.54mm_Vertical"
 			(at 261.62 34.29 0)
 			(hide yes)
@@
 			)
 		)
-		(property "Footprint" ""
+		(property "Footprint" "Resistor_SMD:R_0805_2012Metric"
 			(at 91.44 133.858 90)
 			(hide yes)
@@
 			)
 		)
-		(property "Footprint" ""
+		(property "Footprint" "Connector_PinSocket_2.54mm:PinSocket_1x08_P2.54mm_Vertical"
 			(at 189.23 34.29 0)
 			(hide yes)
@@
 			)
 		)
-		(property "Footprint" ""
+		(property "Footprint" "Connector_PinSocket_2.54mm:PinSocket_1x08_P2.54mm_Vertical"
 			(at 163.83 34.29 0)
 			(hide yes)
@@
 			)
 		)
-		(property "Footprint" ""
+		(property "Footprint" "Resistor_SMD:R_0805_2012Metric"
 			(at 91.44 138.938 90)
 			(hide yes)
@@
 			)
 		)
-		(property "Footprint" ""
+		(property "Footprint" "Connector_PinSocket_2.54mm:PinSocket_1x08_P2.54mm_Vertical"
 			(at 260.35 78.74 0)
 			(hide yes)
@@
 			)
 		)
-		(property "Footprint" ""
+		(property "Footprint" "Resistor_SMD:R_0805_2012Metric"
 			(at 91.44 141.478 90)
 			(hide yes)
@@
 			)
 		)
-		(property "Footprint" ""
+		(property "Footprint" "Capacitor_SMD:C_0805_2012Metric"
 			(at 106.68 147.6248 0)
 			(hide yes)
@@
 			)
 		)
-		(property "Footprint" ""
+		(property "Footprint" "Capacitor_SMD:C_0805_2012Metric"
 			(at 82.55 106.9848 0)
 			(hide yes)
@@
 			)
 		)
-		(property "Footprint" ""
+		(property "Footprint" "Capacitor_SMD:C_0805_2012Metric"
 			(at 104.4448 96.52 0)
 			(hide yes)
@@
 			)
 		)
-		(property "Footprint" ""
+		(property "Footprint" "Resistor_SMD:R_0805_2012Metric"
 			(at 116.84 160.528 90)
 			(hide yes)
@@
 			)
 		)
-		(property "Footprint" ""
+		(property "Footprint" "Connector_PinSocket_2.54mm:PinSocket_1x08_P2.54mm_Vertical"
 			(at 162.56 78.74 0)
 			(hide yes)
@@
 			)
 		)
-		(property "Footprint" ""
+		(property "Footprint" "Connector_PinSocket_2.54mm:PinSocket_1x08_P2.54mm_Vertical"
 			(at 212.09 78.74 0)
 			(hide yes)
@@
 			)
 		)
-		(property "Footprint" ""
+		(property "Footprint" "Capacitor_SMD:C_0805_2012Metric"
 			(at 32.0548 17.78 0)
 			(hide yes)
@@
 			)
 		)
-		(property "Footprint" ""
+		(property "Footprint" "Resistor_SMD:R_0805_2012Metric"
 			(at 116.84 157.988 90)
 			(hide yes)
@@
 			)
 		)
-		(property "Footprint" ""
+		(property "Footprint" "Resistor_SMD:R_0805_2012Metric"
 			(at 100.33 66.548 90)
 			(hide yes)
@@
 			)
 		)
-		(property "Footprint" ""
+		(property "Footprint" "Resistor_SMD:R_0805_2012Metric"
 			(at 91.44 136.398 90)
 			(hide yes)
@@
 			)
 		)
-		(property "Footprint" ""
+		(property "Footprint" "Connector_PinSocket_2.54mm:PinSocket_1x08_P2.54mm_Vertical"
 			(at 187.96 78.74 0)
 			(hide yes)
@@
 			)
 		)
-		(property "Footprint" ""
+		(property "Footprint" "Connector_PinSocket_2.54mm:PinSocket_1x08_P2.54mm_Vertical"
 			(at 213.36 34.29 0)
 			(hide yes)
