File: hardware/kicad/power.kicad_sch (KiCad schematic)
At the start: 16 parts, among them J1 Barrel_Jack, Q1 PMOS, Q3 2N3904, U3 AMS1117-3.3

Commit message: chore: KiCad 회로도 최신 변경사항 반영
원본 작업 폴더가 "회로도 편집 완료/20260901_ver01"로 재구성됨(이전 smartvault-pcb-1
경로는 더 이상 존재하지 않음). 하위 시트 6개 전부와 최상위 시트에 실제 설계 변경
있음(DoorRock-drv는 축소, 최상위 시트는 대폭 확장 — 회로가 재구성된 것으로 보임).
PCB 레이아웃 자체는 변경 없음. footprint.xlsx(부품-풋프린트 매핑) 신규 추가.

파일 내부의 프로젝트명 자기참조는 원본 작업 파일명("20260901_ver01")이 아니라
저장소 표준 이름("smartvault")으로 맞춰서 복사 — 작업 폴더 쪽 날짜/버전 파일명
관례를 저장소까지 끌고 오지 않음(git이 버전을 관리).

s_vault.kicad_sym(커스텀 심볼 라이브러리)은 원본 경로에서 찾지 못해 갱신 못함 —
RS485-com/power 시트가 이 라이브러리를 참조하므로, 최신 심볼이 바뀌었다면 다음에
갱신 필요(hardware/README.md에 기록해둠).

Co-Authored-By: Claude Sonnet 5 <noreply@anthropic.com>
Parts:
- C1: value C -> 100uF/25V; footprint (none) -> Capacitor_THT:CP_Radial_D6.3mm_P2.50mm
- C2: value C -> 0.1uF; footprint (none) -> Capacitor_SMD:C_0805_2012Metric
- C3: value C -> 10uF; footprint (none) -> Capacitor_SMD:C_1206_3216Metric
- C4: value C -> 22uF; footprint (none) -> Capacitor_SMD:C_1210_3225Metric
- C5: renamed from C7; value C -> 10uF; footprint (none) -> Capacitor_SMD:C_1206_3216Metric
- C6: renamed from C8; value C -> 22uF; footprint (none) -> Capacitor_SMD:C_1210_3225Metric
- D1: value D -> SS54_5A/40V; footprint (none) -> Diode_SMD:D_SMB
- F1: value Polyfuse -> Polyfuse_2A; footprint (none) -> Fuse:Fuse_1812_4532Metric
- J1: footprint (none) -> Connector_BarrelJack:BarrelJack_CUI_PJ-102AH_Horizontal
- Q1: value PMOS -> PMOSFET; footprint (none) -> Package_TO_SOT_SMD:SOT-23
- Q3: footprint Package_TO_SOT_THT:TO-92_Inline -> Package_TO_SOT_SMD:SOT-23
- R1: value R -> 10K; footprint (none) -> Resistor_SMD:R_0805_2012Metric
- R2: renamed from R3; value R -> 10K; footprint (none) -> Resistor_SMD:R_0805_2012Metric
- renumbered U2 to U1, U3 to U2
Connections:
- net PWR_EN renamed H_Reset
Other:
- note removed: "sheet2 to 12V/5V SW"
- note removed: "sheet4 WatchDog"
- moved on the sheet: U1
